Commit message: Changed URDF Correctly mapped

File: description/robot_core.xacro (robot description, xacro)
@@ -28,13 +28,13 @@
     <link name="base_footprint">
     </link>
-    <!-- Chasis Link -->
+    <!-- Chassis Link -->
     <joint name="chassis_joint" type="fixed">
         <parent link="base_link"/>
         <child link="chassis"/>
-        <origin xyz="-0.035 0 0"/>
+        <origin xyz="0.035 0 0"/>
     </joint>
     <link name="chassis">
         <visual>
-        	<origin xyz="0.165 0 0.075"/>
+        	<origin xyz="-0.165 0 0.075"/>
             <geometry>
                 <box size="0.33 0.25 0.15"/>
@@ -43,5 +43,5 @@
         </visual>
         <collision>
-            <origin xyz="0.165 0 0.075"/>
+            <origin xyz="-0.165 0 0.075"/>
             <geometry>
                 <box size="0.33 0.25 0.15"/>
@@ -49,5 +49,5 @@
         </collision>
         <xacro:inertial_box mass="3" x="0.33" y="0.24" z="0.15">
-            <origin xyz="0.165 0 0.075" rpy="0 0 0"/>
+            <origin xyz="-0.165 0 0.075" rpy="0 0 0"/>
         </xacro:inertial_box>
     </link>
@@ -60,5 +60,5 @@
         <child link="left_wheel"/>
         <origin xyz="0 0.145 0" rpy="-${pi/2} 0 0" />
-        <axis xyz="0 0 -1"/>
+        <axis xyz="0 0 1"/>
     </joint>
      <!-- length here is the thickness of the wheel -->
@@ -87,5 +87,5 @@
         <child link="right_wheel"/>
         <origin xyz="0 -0.145 0" rpy="${pi/2} 0 0" />
-        <axis xyz="0 0 1"/>
+        <axis xyz="0 0 -1"/>
     </joint>
     <link name="right_wheel">
@@ -112,5 +112,5 @@
         <parent link="chassis"/>
         <child link="caster_wheel"/>
-        <origin xyz="0.25 0 0"/>
+        <origin xyz="-0.25 0 0"/>
     </joint>
     <link name="caster_wheel">
