Commit message: Completed fine tuning Error with Gazebo params yaml file

File: description/robot.urdf.xacro (robot description, xacro)
@@ -1,11 +1,8 @@
 <?xml version="1.0"?>
 <robot xmlns:xacro="http://www.ros.org/wiki/xacro"  name="robot">
-    <!-- <xacro:arg name="use_ros2_control" default="true"/> -->
+    <xacro:arg name="use_ros2_control" default="true"/>
 	<!-- <xacro:arg name="sim_mode" default="false"/> -->
     <xacro:include filename="robot_core.xacro" />
-    <!-- <xacro:include filename="gazebo_control.xacro" /> -->
     <xacro:include filename="lidar.xacro" />
-    <xacro:include filename="ros2_control.xacro"/>
-    <!--
     <xacro:if value="$(arg use_ros2_control)">
         <xacro:include filename="ros2_control.xacro"/>
@@ -14,4 +11,3 @@
         <xacro:include filename="gazebo_control.xacro" />
     </xacro:unless>
-    -->
 </robot>

File: description/robot_core.xacro (robot description, xacro)
@@ -72,5 +72,5 @@
         <collision>
             <geometry>
-                <cylinder radius="0.03" length="0.04"/>
+                <sphere radius="0.03"/>
             </geometry>
         </collision>
@@ -98,5 +98,5 @@
         <collision>
             <geometry>
-                <cylinder radius="0.03" length="0.04"/>
+                <sphere radius="0.03"/>
             </geometry>
         </collision>
